Commit message: Refactor gripper configuration and launch files for dual support; add README documentation

File: robotiq_description/urdf/2f_85.ros2_control.xacro (robot description, xacro)
@@ -47,13 +47,12 @@
             <!-- Joint interfaces -->
             <!-- With Gazebo or Hardware, they handle mimic joints, so we only need this command interface activated -->
-            <!-- We publish joint states: position, velocity, effort and object_detection_status -->
             <joint name="${prefix}robotiq_85_left_knuckle_joint">
                 <command_interface name="position" />
+                <!-- <command_interface name="effort" />
+                <command_interface name="velocity" /> -->
                 <state_interface name="position">
                     <param name="initial_value">${gripper_closed_position}</param>
                 </state_interface>
                 <state_interface name="velocity"/>
-                <state_interface name="effort"/>
-                <state_interface name="object_detection_status"/>
             </joint>
             <!-- When simulating we need to include the rest of the gripper joints -->

File: robotiq_description/urdf/robotiq_2f_85_gripper.urdf.xacro (robot description, xacro)
@@ -4,8 +4,9 @@
     <xacro:arg name="use_fake_hardware" default="true" />
     <xacro:arg name="com_port" default="/dev/ttyUSB0" />
+    <xacro:arg name="prefix" default="" />
     <!-- Import macros -->
     <xacro:include filename="$(find robotiq_description)/urdf/robotiq_2f_85_macro.urdf.xacro" />
-    <link name="world" />
-    <xacro:robotiq_gripper name="RobotiqGripperHardwareInterface" prefix="" parent="world" use_fake_hardware="$(arg use_fake_hardware)" com_port="$(arg com_port)">
+    <link name="$(arg prefix)wrist_3_link" />
+    <xacro:robotiq_gripper name="RobotiqGripperHardwareInterface" prefix="$(arg prefix)" parent="$(arg prefix)wrist_3_link" use_fake_hardware="$(arg use_fake_hardware)" com_port="$(arg com_port)">
         <origin xyz="0 0 0" rpy="0 0 0" />
     </xacro:robotiq_gripper>
